File: DriverConSensorTPFINAL/DriverConSensor.sch (KiCad schematic (older format))
At the start: 51 parts, among them J1 Pulsador1, J2 Pulsador2, J3 Conect_M1, J4 Conect_M2, J5 +12V, J6 Contacto1, J7 GND, K1 SANYOU_SRD_Form_C, K2 SANYOU_SRD_Form_C, K3 SANYOU_SRD_Form_C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

Commit message: actual6
Parts:
- removed U2: L78L05_SO8, Package_SO:SOIC-8_3.9x4.9mm_P1.27mm, symbol Regulator_Linear:L78L05_SO8
- added U2: L78L05_TO92, Package_TO_SOT_THT:TO-92_Inline, symbol Regulator_Linear:L78L05_TO92
- C1: footprint Capacitor_THT:C_Disc_D9.0mm_W2.5mm_P5.00mm -> Capacitor_THT:C_Disc_D3.8mm_W2.6mm_P2.50mm
- C10, C2, C3, C4, C5, C6, C9: footprint (none) -> Capacitor_THT:C_Disc_D3.8mm_W2.6mm_P2.50mm
- C7, C8: footprint (none) -> Capacitor_THT:C_Radial_D6.3mm_H11.0mm_P2.50mm
- J1: value Pulsador1 -> PULS1; footprint (none) -> Connector_Wire:SolderWirePad_1x01_Drill1.2mm
- J2: value Pulsador2 -> PULS2; footprint (none) -> Connector_Wire:SolderWirePad_1x01_Drill1.2mm
- J3: value Conect_M1 -> MotorT2; footprint (none) -> Connector_Wire:SolderWirePad_1x01_Drill2mm
- J4: value Conect_M2 -> MotorT1; footprint (none) -> Connector_Wire:SolderWirePad_1x01_Drill2mm
- J5: value +12V -> VIn+12; footprint (none) -> Connector_Wire:SolderWirePad_1x01_Drill2mm
- J6: value Contacto1 -> Contac12V; footprint (none) -> Connector_Wire:SolderWirePad_1x01_Drill1.2mm
- J7: footprint (none) -> Connector_Wire:SolderWirePad_1x01_Drill2mm
- K1: value SANYOU_SRD_Form_C -> Switch de Encendido
- K2, K3: value SANYOU_SRD_Form_C -> FRS10CS10-12V
- Q1, Q2: footprint Package_TO_SOT_THT:TO-92_Inline -> Package_TO_SOT_THT:TO-92_Inline_Wide
- R1, R10, R11, R12, R13, R14, R15, R16, R17, R2, R3, R4, R5, R6, R7, R8, R9: footprint (none) -> Resistor_THT:R_Axial_DIN0204_L3.6mm_D1.6mm_P7.62mm_Horizontal
- SW1: footprint (none) -> Button_Switch_THT:SW_DIP_SPSTx06_Slide_6.7x16.8mm_W7.62mm_P2.54mm_LowProfile
Connections:
- wire segments 177 -> 185
Other:
- note added: "Activa todo el dispositivo, \npermitiendo alimentar \nlas proximas etapas\n con los 12v"
- note added: "El Pic por un lado mueve el motor hacia \nun lado u hacia el otro según las entradas\nen pulsador 1 o pulsador 2, y segun el \nsensor de corriente lo frena enviando\nlas señales correspondiente a las \nbases de los transistores.\n"
- note added: "El código activa o \ndesactiva los \nrelay"
- note added: "El valor de corriente \nsensador y ajustado en\nel dipswitch \nva hacia el microcontrolador\n"
- note added: "Esta entrada viene de un\npulsador que al ser pulsado\nes puesto a tierra\nactivando logicamente a\nGP1\n\n"
- note added: "Esta entrada viene de un\npulsador que al ser pulsado\nes puesto a tierra\nactivando logicamente a\nGP2\n"
- note added: "REGULADOR DE 5V\n"
- note added: "Si ambos Relay están en GND (Normal Cerrado) \nestán desactivados los bornes del motor.\n En cuanto se activa uno (12V) el otro \npermanece desactivado(GND) por lo tanto \nel motor gira en una dirección y vicecersa \npara cambiar de dirección."
- note removed: "El valor de corriente \nsensador y ajustado en\nel dipswitch \nva hacia el micro"
- moved on the sheet: C1, C10, C2, C3, C4, C5, C6, C7, C8, C9, D10, D3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
