File: DriverConSensorTPFINAL/DriverConSensor.kicad_pcb (KiCad board)
At the start: 2 copper layers, 77 x 67 mm, 51 parts, among them J1 PULS1, J2 PULS2, J3 MotorT2, J4 MotorT1, J5 VIn+12, J6 Contac12V, J7 GND, K1 Switch de Encendido, K2 FRS10CS10-12V, K3 FRS10CS10-12V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

Commit message: actual2
Parts:
- moved R2 0.59 mm to (187.8, 107.4)
- moved R3 0.59 mm to (187.8, 103.4)
- moved D3 0.59 mm to (180.1, 119.7)
- moved D5 0.59 mm to (180.1, 115.0)
- moved R1 0.59 mm to (180.1, 111.4)
Routing:
- net GND: track 228.2 -> 239.4 mm
- net +5V: track 216.4 -> 221.3 mm
- net Net-(D6-Pad2): track 18.1 -> 13.3 mm
- net Net-(D5-Pad2): track 17.8 -> 13.3 mm
- added copper zone on B.Cu, net GND

Commit message: actual3
Routing:
- net GND: track 239.4 -> 294.8 mm
Changed lines of the file:
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@@
     (thickness 1.6)
     (drawings 8)
-    (tracks 338)
+    (tracks 354)
     (zones 0)
     (modules 51)
@@
   (gr_line (start 190 130) (end 190 63) (layer Edge.Cuts) (width 0.05))
   (gr_line (start 113 130) (end 190 130) (layer Edge.Cuts) (width 0.05))
+  (segment (start 161.05 115.91) (end 161.05 114.26494) (width 0.6) (layer F.Cu) (net 1))
   (segment (start 126.375 97.75) (end 123.96707 97.75) (width 0.6) (layer B.Cu) (net 1))
   (segment (start 186.9 94.72) (end 188.3 93.32) (width 0.8) (layer B.Cu) (net 1))
@@
   (segment (start 161.775 124.425) (end 160.975001 125.224999) (width 1) (layer B.Cu) (net 1))
   (segment (start 160.975001 125.224999) (end 160.975001 126.875001) (width 1) (layer B.Cu) (net 1))
+  (segment (start 149.935 78.97) (end 145.725 78.97) (width 1) (layer F.Cu) (net 1))
+  (segment (start 157.555 71.35) (end 149.935 78.97) (width 1) (layer F.Cu) (net 1))
+  (segment (start 183.6 95.85137) (end 183.6 94.72) (width 1) (layer F.Cu) (net 1))
+  (segment (start 180.25137 99.2) (end 183.6 95.85137) (width 1) (layer F.Cu) (net 1))
+  (segment (start 172.2 99.2) (end 180.25137 99.2) (width 1) (layer F.Cu) (net 1))
+  (segment (start 171.28 91.8) (end 175.98 87.1) (width 1) (layer F.Cu) (net 1))
+  (segment (start 170.15 91.8) (end 171.28 91.8) (width 1) (layer F.Cu) (net 1))
+  (segment (start 170.15 91.8) (end 170.15 94.14) (width 1) (layer F.Cu) (net 1))
+  (segment (start 172.2 96.19) (end 172.2 99.2) (width 1) (layer F.Cu) (net 1))
+  (segment (start 170.15 94.14) (end 172.2 96.19) (width 1) (layer F.Cu) (net 1))
+  (segment (start 161.775 124.425) (end 161.775 118.515) (width 1) (layer F.Cu) (net 1))
+  (segment (start 160.699999 116.130001) (end 160.699999 116.108112) (width 1) (layer F.Cu) (net 1))
+  (segment (start 161.775 118.515) (end 160.699999 117.439999) (width 1) (layer F.Cu) (net 1))
+  (segment (start 160.699999 117.439999) (end 160.699999 116.130001) (width 1) (layer F.Cu) (net 1))
   (segment (start 120.575 107.425) (end 120.575 105.201998) (width 1) (layer B.Cu) (net 2))
   (segment (start 117.375 110.625) (end 120.575 107.425) (width 1) (layer B.Cu) (net 2))
@@
   (segment (start 175.964937 126.475061) (end 172.31403 126.475061) (width 0.8) (layer B.Cu) (net 2))
   (segment (start 178.074999 124.364999) (end 175.964937 126.475061) (width 0.8) (layer B.Cu) (net 2))
+  (segment (start 126.07498 102.20002) (end 126.07498 101.83002) (width 1) (layer B.Cu) (net 2))
   (segment (start 184.800001 98.400001) (end 179.800001 98.400001) (width 1) (layer B.Cu) (net 3))
   (segment (start 185.6 99.2) (end 184.800001 98.400001) (width 1) (layer B.Cu) (net 3) (status 10))

Commit message: actual4
Parts:
- added REF**: SolderWirePad_1x01_Drill1mm, Connector_Wire:SolderWirePad_1x01_Drill1mm, F.Cu at (162.9, 74.7)
- added REF**: SolderWirePad_1x01_Drill1mm, Connector_Wire:SolderWirePad_1x01_Drill1mm, F.Cu at (163.0, 89.1)
- moved R11 6.99 mm to (158.3, 72.6), turned to 90 degrees
- moved D7 6.97 mm to (143.6, 88.6)
- moved D9 6.76 mm to (143.6, 92.5)
- moved C8 4.82 mm to (161.1, 120.8), turned to 270 degrees
- moved D10 4.65 mm to (143.3, 115.9)
- moved C6 3.71 mm to (170.4, 93.0), turned to 90 degrees
- moved C7 2.80 mm to (154.7, 112.8)
- moved R10 2.55 mm to (132.1, 85.5)
- moved R8 2.48 mm to (161.1, 106.0)
- moved R9 2.22 mm to (158.2, 97.7)
- moved R16 1.92 mm to (166.9, 70.5)
- moved SW1 1.92 mm to (185.9, 81.5)
- moved R15 1.92 mm to (166.9, 74.1)
- moved R13 1.92 mm to (166.8, 81.1)
- moved R14 1.92 mm to (166.8, 77.4)
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Routing:
- net GND: track 294.8 -> 262.1 mm
- net /GP5(PIN3PIC): track 39.6 -> 32.4 mm
- net Net-(R13-Pad1): track 136.9 -> 130.8 mm
- net Net-(D7-Pad2): track 87.1 -> 82.9 mm
- net /Relay2y3_NA: track 93.7 -> 89.5 mm
- net Net-(C5-Pad2): track 3.36 -> 6.98 mm
- net +12V: track 53.6 -> 50.1 mm
- net Net-(C4-Pad1): track 7.49 -> 4.30 mm
- net /GPIO0(PIN7PIC): track 31.9 -> 29.4 mm
- net Net-(C4-Pad2): track 16.4 -> 14.5 mm
- net Net-(C2-Pad2): track 20.8 -> 19.0 mm
- net +5V: track 221.6 -> 222.7 mm
- net /GP4(PIN2PIC): track 22.5 -> 21.7 mm
Other:
- outline, holes or cut-outs redrawn

Commit message: actual5
Parts:
- removed the REF** at (162.9, 74.7)
- removed the REF** at (163.0, 89.1)
- added REF**: SolderWirePad_1x01_Drill0.8mm, Connector_Wire:SolderWirePad_1x01_Drill0.8mm, F.Cu at (161.9, 73.6)
- added REF**: SolderWirePad_1x01_Drill0.8mm, Connector_Wire:SolderWirePad_1x01_Drill0.8mm, F.Cu at (161.9, 86.8)
- moved K2 1.00 mm to (133.9, 75.7)
- moved R10 0.95 mm to (132.7, 86.3)
Routing:
- net GND: track 262.1 -> 281.4 mm
- net Net-(D7-Pad2): track 82.9 -> 77.2 mm
- net /Relay2y3_NA: track 89.5 -> 93.6 mm
- net Net-(C5-Pad1): track 13.7 -> 15.4 mm
- net Net-(R13-Pad1): track 130.8 -> 129.3 mm
- net Net-(D7-Pad1): track 38.6 -> 37.6 mm
Other:
- net class c added: clearance 0.4, trace_width 0.8, via_dia 1, via_drill 0.8
- board text added: "El pad GND1 y GND2 es para colocar un cable e dichos lugares para reforzar la uio de amas masas, que se realiza e el relleno de cobre por un lugar estrecho"

Commit message: actual7
Routing:
- net GND: track 281.4 -> 277.3 mm
- net Net-(D7-Pad1): track 37.6 -> 37.0 mm
- net +5V: track 222.7 -> 222.1 mm
Other:
- board text added: "El pad GND1 y GND2 es para colocar un cable en dichos lugares para reforzar la union de ambas masas, que se realiza en el relleno de cobre por un lugar estrecho"
- board text removed: "El pad GND1 y GND2 es para colocar un cable e dichos lugares para reforzar la uio de amas masas, que se realiza e el relleno de cobre por un lugar estrecho"
