File: TPFINAL2NOV19/DriverConSensor.kicad_pcb (KiCad board)
At the start: 2 copper layers, 77 x 67 mm, 53 parts, among them J1 PULS1, J2 PULS2, J3 MotorT2, J4 MotorT1, J5 VIn+12, J6 Contac12V, J7 GND, K1 Switch de Encendido, K2 FRS10CS10-12V, K3 FRS10CS10-12V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

Commit message: PCb
Parts:
- C9: moved to F.Cu
- U3: moved to B.Cu
- moved C1 20.5 mm to (131.2, 125.8), turned to 270 degrees
- moved C9 3.95 mm to (116.9, 87.6), turned to 0 degrees
Routing:
- net GND: track 277.3 -> 287.6 mm
- net +5V: track 222.1 -> 213.3 mm
- net Net-(C9-Pad1): track 13.1 -> 18.4 mm
- net Net-(R13-Pad1): track 129.3 -> 125.0 mm
- net /Relay2y3_NA: track 93.6 -> 90.1 mm
Other:
- board text added: "Los Capacitores C6, C3 y C9 fueron modificados sus huellas para facilitar el diseño ya que en la implemetación se colocarán las patas en esas medidas, siendo esto posible por la flexibilidad de las mismas"

Commit message: PCB_casi_listo2
Other:
- board text added: "Me FALTA CORREGIR ACA QUE EL RELLENO DE COBRE ME INVADIO ESTA ZONA"
Changed lines of the file:
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@@
   (general
     (thickness 1.6)
-    (drawings 11)
+    (drawings 12)
     (tracks 371)
     (zones 0)
@@
     )
   )
+  (gr_text "Me FALTA CORREGIR ACA QUE EL\n RELLENO DE COBRE ME INVADIO ESTA ZONA" (at 53.625 99.25) (layer B.Cu)
+    (effects (font (size 1.5 1.5) (thickness 0.3)) (justify left))
+  )
   (gr_text "Los Capacitores C6, C3 y C9 fueron modificados sus huellas\n para facilitar el diseño ya que en la implemetación se colocarán\n las patas en esas medidas, siendo esto posible por la\n flexibilidad de las mismas" (at 199.725 76.825) (layer B.Cu)

Commit message: PCB_casi_listo3
Parts:
- U2: value L78L05 -> L78L05_TO92
Connections:
- U3 pad 1: +12V -> /Relay2y3_NA
- U3 pad 2: +12V -> /Relay2y3_NA
- U3 pad 3: /Relay2y3_NA -> +12V
- U3 pad 4: /Relay2y3_NA -> +12V
Routing:
- net Net-(C9-Pad1): track 18.4 -> 20.4 mm
- net Net-(R13-Pad1): track 125.0 -> 125.5 mm

Commit message: PCB_casi_listo4
Parts:
- C3, C6, C9: footprint Capacitor_THT:C_Disc_D3.8mm_W2.6mm_P2.50mm -> Capacitor_THT:C_Disc_D5.0mm_W2.5mm_P5.00mm
Other:
- board text removed: "Me FALTA CORREGIR ACA QUE EL RELLENO DE COBRE ME INVADIO ESTA ZONA"

Commit message: PCB_casi_listo5
Routing:
- net +5V: track 213.5 -> 214.2 mm
Changed lines of the file:
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@@
   )
   (setup
-    (last_trace_width 0.6)
+    (last_trace_width 0.8)
     (user_trace_width 0.6)
     (user_trace_width 0.8)
@@
       (effects (font (size 1 1) (thickness 0.15)))
     )
-    (fp_text user %R (at 0 0) (layer F.Fab)
+    (fp_text user GND (at 0 0) (layer F.Fab)
       (effects (font (size 1 1) (thickness 0.15)))
     )
@@
     (fp_line (start -1.5 -1.5) (end -1.5 1.5) (layer F.CrtYd) (width 0.05))
     (fp_line (start -1.5 -1.5) (end 1.5 -1.5) (layer F.CrtYd) (width 0.05))
-    (fp_text user %R (at 0 0) (layer F.Fab)
+    (fp_text user GND (at 0 0) (layer F.Fab)
       (effects (font (size 1 1) (thickness 0.15)))
     )
@@
       (effects (font (size 1 1) (thickness 0.15)))
     )
-    (fp_text user %R (at 1.25 0 90) (layer F.Fab)
+    (fp_text user %R (at 1.25 0 180) (layer F.Fab)
       (effects (font (size 0.76 0.76) (thickness 0.114)))
     )
@@
     (fp_line (start 3.55 1.55) (end 3.55 -1.55) (layer F.CrtYd) (width 0.05))
     (fp_line (start 3.55 -1.55) (end -1.05 -1.55) (layer F.CrtYd) (width 0.05))
-    (fp_text user %R (at 1.25 0 90) (layer F.Fab)
+    (fp_text user %R (at 1.25 0 180) (layer F.Fab)
       (effects (font (size 0.76 0.76) (thickness 0.114)))
     )
@@
       (effects (font (size 1 1) (thickness 0.15)))
     )
-    (fp_text user %R (at 0 0) (layer F.Fab)
+    (fp_text user M1 (at 0 0) (layer F.Fab)
       (effects (font (size 1 1) (thickness 0.15)))
     )
@@
     (fp_line (start -2.75 -2.75) (end -2.75 2.75) (layer F.CrtYd) (width 0.05))
     (fp_line (start -2.75 -2.75) (end 2.75 -2.75) (layer F.CrtYd) (width 0.05))
-    (fp_text user %R (at 0 0) (layer F.Fab)
+    (fp_text user M2 (at 0 0) (layer F.Fab)
       (effects (font (size 1 1) (thickness 0.15)))
     )
@@
       (effects (font (size 1 1) (thickness 0.15)))
     )
-    (fp_text user %R (at 0 0) (layer F.Fab)
+    (fp_text user 12v (at 0 0) (layer F.Fab)
       (effects (font (size 1 1) (thickness 0.15)))
     )
@@
       (effects (font (size 0.8 0.8) (thickness 0.1)))
     )
-    (fp_text user %R (at 0 0) (layer F.Fab)
-      (effects (font (size 1 1) (thickness 0.15)))
+    (fp_text user Cont12V (at 0 0) (layer F.Fab)
+      (effects (font (size 0.8 0.8) (thickness 0.1)))
     )
     (fp_line (start -2.25 -2.25) (end 2.25 -2.25) (layer F.CrtYd) (width 0.05))
@@
     (fp_line (start -2.75 -2.75) (end -2.75 2.75) (layer F.CrtYd) (width 0.05))
     (fp_line (start -2.75 -2.75) (end 2.75 -2.75) (layer F.CrtYd) (width 0.05))
-    (fp_text user %R (at 0 0) (layer F.Fab)
+    (fp_text user GND (at 0 0) (layer F.Fab)
       (effects (font (size 1 1) (thickness 0.15)))
     )
@@
   (segment (start 167.08 103.3) (end 162.70001 107.67999) (width 1) (layer B.Cu) (net 2))
   (segment (start 162.70001 107.67999) (end 162.70001 109.20001) (width 1) (layer B.Cu) (net 2))
-  (segment (start 176.600001 98.300001) (end 175.712699 97.412699) (width 0.8) (layer B.Cu) (net 2))
-  (segment (start 182.055001 105.325001) (end 182.055001 108.456999) (width 0.8) (layer B.Cu) (net 2))
-  (segment (start 182.055001 108.456999) (end 180.987001 109.524999) (width 0.8) (layer B.Cu) (net 2))
-  (segment (start 180.987001 109.524999) (end 179.187753 109.524999) (width 0.8) (layer B.Cu) (net 2))
-  (segment (start 180.155 103.425) (end 182.055001 105.325001) (width 0.8) (layer B.Cu) (net 2))
-  (segment (start 179.187753 109.524999) (end 176.600001 106.937247) (width 0.8) (layer B.Cu) (net 2))
-  (segment (start 176.600001 106.937247) (end 176.600001 98.300001) (width 0.8) (layer B.Cu) (net 2))
-  (segment (start 167.691992 109.20001) (end 162.70001 109.20001) (width 0.8) (layer B.Cu) (net 2))
-  (segment (start 168.980001 107.912001) (end 167.691992 109.20001) (width 0.8) (layer B.Cu) (net 2))
-  (segment (start 168.980001 107.221333) (end 168.980001 107.912001) (width 0.8) (layer B.Cu) (net 2))
-  (segment (start 170.40001 105.801324) (end 168.980001 107.221333) (width 0.8) (layer B.Cu) (net 2))
-  (segment (start 170.400011 101.399989) (end 170.40001 105.801324) (width 0.8) (layer B.Cu) (net 2))
-  (segment (start 171.700001 100.099999) (end 170.400011 101.399989) (width 0.8) (layer B.Cu) (net 2))
-  (segment (start 171.700001 98.499999) (end 171.700001 100.099999) (width 0.8) (layer B.Cu) (net 2))
-  (segment (start 172.787301 97.412699) (end 171.700001 98.499999) (width 0.8) (layer B.Cu) (net 2))
-  (segment (start 175.712699 97.412699) (end 172.787301 97.412699) (width 0.8) (layer B.Cu) (net 2))
   (segment (start 160.300001 120.000001) (end 158.425001 120.000001) (width 1) (layer B.Cu) (net 2))
   (segment (start 161.1 120.8) (end 160.300001 120.000001) (width 1) (layer B.Cu) (net 2))
@@
   (segment (start 127.53994 97.745) (end 128.45001 98.65507) (width 0.6) (layer B.Cu) (net 2))
   (segment (start 126.35 97.745) (end 127.53994 97.745) (width 0.6) (layer B.Cu) (net 2))
+  (segment (start 168.980001 107.221333) (end 168.980001 107.912001) (width 0.8) (layer B.Cu) (net 2))
+  (segment (start 170.40001 105.801324) (end 168.980001 107.221333) (width 0.8) (layer B.Cu) (net 2))
+  (segment (start 170.400011 101.399989) (end 170.40001 105.801324) (width 0.8) (layer B.Cu) (net 2))
+  (segment (start 171.700001 100.099999) (end 170.400011 101.399989) (width 0.8) (layer B.Cu) (net 2))
+  (segment (start 173.25 96.95) (end 171.700001 98.499999) (width 0.8) (layer B.Cu) (net 2))
+  (segment (start 182.055001 105.325001) (end 182.055001 108.456999) (width 0.8) (layer B.Cu) (net 2))
+  (segment (start 168.980001 107.912001) (end 167.691992 109.20001) (width 0.8) (layer B.Cu) (net 2))
+  (segment (start 180.155 103.425) (end 182.055001 105.325001) (width 0.8) (layer B.Cu) (net 2))
+  (segment (start 167.691992 109.20001) (end 162.70001 109.20001) (width 0.8) (layer B.Cu) (net 2))
+  (segment (start 176.600001 97.825001) (end 175.725 96.95) (width 0.8) (layer B.Cu) (net 2))
+  (segment (start 180.987001 109.524999) (end 179.187753 109.524999) (width 0.8) (layer B.Cu) (net 2))
+  (segment (start 171.700001 98.499999) (end 171.700001 100.099999) (width 0.8) (layer B.Cu) (net 2))
+  (segment (start 179.187753 109.524999) (end 176.600001 106.937247) (width 0.8) (layer B.Cu) (net 2))
+  (segment (start 175.725 96.95) (end 173.25 96.95) (width 0.8) (layer B.Cu) (net 2))
+  (segment (start 182.055001 108.456999) (end 180.987001 109.524999) (width 0.8) (layer B.Cu) (net 2))
+  (segment (start 176.600001 106.937247) (end 176.600001 97.825001) (width 0.8) (layer B.Cu) (net 2))
   (segment (start 178.52 97.12) (end 178.52 94.72) (width 1) (layer B.Cu) (net 3) (status 20))
   (segment (start 180.59 99.19) (end 178.52 97.12) (width 1) (layer B.Cu) (net 3))

Commit message: PCB
Parts:
- moved J5 0.40 mm to (116.4, 117.5)
- renumbered REF** to GND
Other:
- board text added: "Industria Argentina"
- board text added: "JPM"
- board text removed: "Los Capacitores C6, C3 y C9 fueron modificados sus huellas para facilitar el diseño ya que en la implemetación se colocarán las patas en esas medidas, siendo esto posible por la flexibilidad de las mismas"

Commit message: PCB
Parts:
- K1, K2, K3: footprint Relay_THT:Relay_SPDT_SANYOU_SRD_Series_Form_C -> Relay_THT:Relay_SPDT_Omron-G5LE-1
- moved D10 0.78 mm to (144.1, 116.0)
- moved J3 0.55 mm to (144.8, 99.2)
- moved K3 0.53 mm to (139.2, 99.1), turned to 270 degrees
- moved D8 0.51 mm to (136.9, 88.9)
- moved D7 0.20 mm to (143.6, 88.4)
- turned K1 to 90 degrees
- turned K2 to 270 degrees
Routing:
- net Net-(C4-Pad2): track 14.5 -> 16.0 mm

Commit message: PCB
Parts:
- moved C1 1.07 mm to (131.4, 126.8), turned to 180 degrees
- moved C4 0.46 mm to (155.6, 100.7)
Routing:
- net GND: track 287.8 -> 253.1 mm
- net Net-(C4-Pad2): track 16.0 -> 17.2 mm
- net +5V: track 214.2 -> 214.7 mm
Other:
- board text added: "Las pistas que estan marcadas con máscara antisoldante quedan libres para ser reforzadas con estaño"
- board text added: "Versión 1.0 - 2019"
