File: TPFINAL2NOV19/DriverConSensor.kicad_pcb (KiCad board)
At the start: 2 copper layers, 77 x 67 mm, 53 parts, among them J1 PULS1, J2 PULS2, J3 MotorT2, J4 MotorT1, J5 VIn+12, J6 Contac12V, J7 GND, K1 Switch de Encendido, K2 FRS10CS10-12V, K3 FRS10CS10-12V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

Commit message: PCB
Other:
- board text added: "Grillas: 1 mm, 0,5 mm , 0,10 mm Margen: 0.3 mm Pista: 0.6 mm, 0.8mm, 1mm, 2 mm, 3mm Dist. a borde: 0.40 mm Terminacion: Estaño Plomo (Sn/Pb)"
Changed lines of the file:
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@@
   (general
     (thickness 1.6)
-    (drawings 30)
+    (drawings 31)
     (tracks 377)
     (zones 0)
@@
     (visible_elements FFFDFF7F)
     (pcbplotparams
-      (layerselection 0x31170_ffffffff)
+      (layerselection 0x11060_ffffffff)
       (usegerberextensions false)
       (usegerberattributes false)
@@
     )
   )
-  (gr_text "Las pistas que estan marcadas con máscara antisoldante \nquedan libres para ser reforzadas con estaño" (at 233.39 76.15) (layer F.CrtYd)
-    (effects (font (size 1.5 1.5) (thickness 0.3)))
+  (gr_text "Grillas: 1 mm, 0,5 mm , 0,10 mm\nMargen: 0.3 mm\nPista: 0.6 mm, 0.8mm, 1mm, 2 mm, 3mm\nDist. a borde: 0.40 mm\nTerminacion: Estaño Plomo (Sn/Pb)" (at 203.17 90.74) (layer F.CrtYd)
+    (effects (font (size 1.5 1.5) (thickness 0.3)) (justify left))
+  )
+  (gr_text "Las pistas que estan marcadas con máscara antisoldante \nquedan libres para ser reforzadas con estaño" (at 203.61 75.79) (layer F.CrtYd)
+    (effects (font (size 1.5 1.5) (thickness 0.3)) (justify left))
   )
   (gr_line (start 139.2 77.575) (end 135.8 77.625) (layer B.Mask) (width 3))
@@
     (effects (font (size 1.8 1.8) (thickness 0.25)))
   )
-  (gr_text "El pad GND1 y GND2 es para colocar un cable en dichos \nlugares para reforzar la union de ambas masas, que se \nrealiza en el relleno de cobre por un lugar estrecho" (at 200.25 63.775) (layer F.CrtYd)
+  (gr_text "El pad GND1 y GND2 es para colocar un cable en dichos \nlugares para reforzar la union de ambas masas, que se \nrealiza en el relleno de cobre por un lugar estrecho" (at 203.17 64.35) (layer F.CrtYd)
     (effects (font (size 1.5 1.5) (thickness 0.3)) (justify left))
   )

Commit message: PCB_Final
Parts:
- moved C4 73.1 mm to (96.8, 57.1), turned to 90 degrees
- moved R9 71.5 mm to (97.6, 59.7), turned to 270 degrees
- moved D8 70.6 mm to (82.7, 43.6)
- moved K3 69.9 mm to (85.8, 54.0)
- moved J3 69.5 mm to (92.1, 54.0)
- moved J7 64.6 mm to (95.1, 42.6)
- moved 1 62.0 mm to (106.7, 58.6)
- moved R8 60.8 mm to (115.6, 65.8)
- moved 1 59.8 mm to (106.6, 50.9)
- moved C8 56.6 mm to (110.4, 95.6)
- moved U2 56.2 mm to (111.9, 89.6)
- moved R2 54.9 mm to (138.7, 82.5)
- moved R11 54.9 mm to (109.2, 48.1)
- moved R12 54.9 mm to (137.7, 61.2)
- moved R3 54.9 mm to (138.7, 78.9)
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- renumbered GND to 1
Connections:
- 1 pad 2: GND -> Net-(R13-Pad1)
- 1 pad 1: GND -> Net-(R13-Pad1)
- C7 pad 1: +12V -> Net-(C7-Pad1)
- D10 pad 1: +12V -> Net-(C7-Pad1)
- J5 pad 1: Net-(J5-Pad1) -> +12V
- K1 pad 1: Net-(J5-Pad1) -> +12V
- K1 pad 3: +12V -> Net-(K1-Pad3)
- U2 pad 3: +12V -> Net-(C7-Pad1)
- U3 pad 3: +12V -> Net-(K1-Pad3)
- U3 pad 4: +12V -> Net-(K1-Pad3)
Routing:
- net GND: track 253.1 -> 86.6 mm
- net +12V: track 50.2 -> 6.70 mm
- net Net-(D7-Pad1): track 37.0 -> 71.0 mm
- net /Relay2y3_NA: track 90.0 -> 117.1 mm
- net +5V: track 214.7 -> 193.6 mm
- net Net-(C7-Pad1): track 0.00 -> 16.0 mm
- net Net-(R13-Pad1): track 125.5 -> 110.1 mm
- net /GP5(PIN3PIC): track 32.4 -> 19.1 mm
- net /GP4(PIN2PIC): track 21.7 -> 8.36 mm
- net Net-(D7-Pad2): track 77.2 -> 85.2 mm
- net Net-(C9-Pad1): track 20.4 -> 13.8 mm
- net Net-(J5-Pad1): track 6.38 -> 0.00 mm
- net Net-(K1-Pad3): track 0.00 -> 5.99 mm
- net Net-(Q2-Pad2): track 6.00 -> 11.5 mm
- net Net-(C4-Pad2): track 17.2 -> 12.6 mm
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Other:
- rule via_min_size: 0.4 -> 0.3
- board text added: "AGUJERO DE SUJECIÓN : Esta placa iria en una caja de plastico que posee dos cilindros pasantes para sostener la misma, que son los dos agujeros representados por circulos. Si queda u zoa fragil como mecionó en la corrección pero es por que el case donde va ir alojada ya esta hecho, se busca reemplazar una placa ya hecha actualmente con las mismas medidas de forma"
- board text added: "CtrlMotVidr Versión 2.0 - Nov2019"
- board text added: "Diseño Argentino"
- board text added: "Grillas: 1 mm, 0,5 mm , 0,10 mm Margen: 0.3 mm Pista: 0.6 mm, 0.8mm, 1mm, 2 mm, 3mm Dist. a borde: 0.40 mm Terminacion: HASL Fabricante: Mayer"
- board text added: "Q1 y Q2; si bien en el esquematico se menciona aclaro aca su función, los mismos estan en paralelo en cuanto a colector-emisor, pero la base de cada uno esta conectada a la salida de los GPIO para que puedan ser activas o desactivados segun una logica que es la siguientes: Cuando se activa un GPIO mueve un relay por donde queda a 12v y de ahi va a lo borne del motor, el otro motor esta al otro re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"
- board text added: "SMD :la razon de uso de un componente SMD es que este modelo en particular es un sensor de corriente de 30A para uso en el rubro automotor solo con encapsulado smd se consigue. No se opto por hacer smd en su totalidad por falta de experiencia, pero se realizará a futuro para una mejora de la presente versión"
- board text removed: "Grillas: 1 mm, 0,5 mm , 0,10 mm Margen: 0.3 mm Pista: 0.6 mm, 0.8mm, 1mm, 2 mm, 3mm Dist. a borde: 0.40 mm Terminacion: Estaño Plomo (Sn/Pb)"
- board text removed: "Industria Argentina"
- board text removed: "Versión 1.0 - 2019"

Commit message: PCB_Final
Parts:
- moved C1 1.40 mm to (104.1, 93.8)
Routing:
- net Net-(D7-Pad1): track 71.0 -> 73.1 mm
- net +5V: track 193.6 -> 195.5 mm
- net Net-(R13-Pad1): track 110.1 -> 108.5 mm
- net Net-(C7-Pad1): track 16.0 -> 17.6 mm
- net GND: track 86.6 -> 85.5 mm
Changed lines of the file:
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@@
     (thickness 1.6)
     (drawings 29)
-    (tracks 319)
+    (tracks 325)
     (zones 0)
     (modules 53)
@@
   )
   (module Capacitor_THT:C_Disc_D3.8mm_W2.6mm_P2.50mm (layer F.Cu)
-    (at 103.05 94.8 90)
+    (at 104.075 93.85 90)
     (descr "C, Disc series, Radial, pin pitch=2.50mm, , diameter*width=3.8*2.6mm^2, Capacitor, http://www.vishay.com/docs/45233/krseries.pdf")
     (tags "C Disc series Radial pin pitch 2.50mm  diameter 3.8mm width 2.6mm Capacitor")
-    (fp_text reference C1 (at 5.175 2.1 180) (layer F.SilkS)
+    (fp_text reference C1 (at 4.625 1.575 180) (layer F.SilkS)
       (effects (font (size 1 1) (thickness 0.15)))
     )
@@
   (gr_line (start 140.925 105.475) (end 140.925 38.475) (layer Edge.Cuts) (width 0.05))
   (gr_line (start 63.925 105.475) (end 140.925 105.475) (layer Edge.Cuts) (width 0.05))
-  (segment (start 67.59999 91.99999) (end 70.31501 94.71501) (width 3) (layer B.Cu) (net 29))
   (segment (start 138.62 101.905) (end 138.62 95.2) (width 1) (layer B.Cu) (net 1) (status 20))
   (segment (start 136.305 70.195) (end 137.695 68.805) (width 1) (layer B.Cu) (net 1) (status 20))
@@
   (segment (start 126.905 62.575) (end 122.225 62.575) (width 1) (layer B.Cu) (net 1) (status 10))
   (segment (start 111.145 54.495) (end 109.125 54.495) (width 1) (layer B.Cu) (net 1) (status 20))
-  (segment (start 103.125 92.275) (end 101.99363 92.275) (width 1) (layer B.Cu) (net 1))
   (segment (start 134.525 62.006998) (end 131.763002 59.245) (width 1) (layer B.Cu) (net 2) (status 10))
   (segment (start 134.525 62.575) (end 134.525 62.006998) (width 1) (layer B.Cu) (net 2) (status 30))
@@
   (segment (start 115.625 84.875) (end 115.725 84.975) (width 1) (layer B.Cu) (net 2))
   (segment (start 115.725 94.874999) (end 114.324999 96.275) (width 1) (layer B.Cu) (net 2))
-  (segment (start 114.324999 96.275) (end 112.025 96.275) (width 1) (layer B.Cu) (net 2))
-  (segment (start 112.025 96.275) (end 111.225001 95.475001) (width 1) (layer B.Cu) (net 2))
-  (segment (start 111.225001 95.475001) (end 109.350001 95.475001) (width 1) (layer B.Cu) (net 2))
   (segment (start 115.725 84.975) (end 115.725 90.075) (width 1) (layer B.Cu) (net 2))
   (segment (start 115.725 90.075) (end 115.725 94.874999) (width 1) (layer B.Cu) (net 2))
@@
   (segment (start 114.0723 89.6258) (end 114.5215 90.075) (width 1) (layer B.Cu) (net 2))
   (segment (start 112.5473 89.6258) (end 114.0723 89.6258) (width 1) (layer B.Cu) (net 2) (status 10))
-  (segment (start 110.1056 94.9) (end 103.05 94.9) (width 1) (layer B.Cu) (net 2))
-  (segment (start 110.4377 95.2321) (end 110.1056 94.9) (width 1) (layer B.Cu) (net 2))
-  (segment (start 101.91863 94.9) (end 103.05 94.9) (width 1) (layer B.Cu) (net 2))
-  (segment (start 78.45 95.11001) (end 78.45 100.9) (width 1) (layer B.Cu) (net 2))
-  (segment (start 78.45 100.9) (end 80.775 103.225) (width 1) (layer B.Cu) (net 2))
-  (segment (start 80.775 103.225) (end 93.775 103.225) (width 1) (layer B.Cu) (net 2))
-  (segment (start 101.15451 94.9) (end 101.91863 94.9) (width 1) (layer B.Cu) (net 2))
-  (segment (start 93.775 103.225) (end 97.835604 99.164396) (width 1) (layer B.Cu) (net 2))
-  (segment (start 97.835604 99.164396) (end 97.835604 98.218906) (width 1) (layer B.Cu) (net 2))
-  (segment (start 97.835604 98.218906) (end 101.15451 94.9) (width 1) (layer B.Cu) (net 2))
   (segment (start 115.025001 41.374999) (end 115.025001 42.520997) (width 0.8) (layer B.Cu) (net 2))
   (segment (start 115.025001 42.520997) (end 114.370998 43.175) (width 0.8) (layer B.Cu) (net 2))
@@
   (segment (start 119.755001 41.615997) (end 119.755001 41.442999) (width 0.8) (layer B.Cu) (net 2))
   (segment (start 119.957002 41.817998) (end 119.755001 41.615997) (width 0.8) (layer B.Cu) (net 2))
+  (segment (start 110.4377 95.2321) (end 109.637701 94.432101) (width 1) (layer B.Cu) (net 2))
+  (segment (start 80.775 103.225) (end 95.125 103.225) (width 1) (layer B.Cu) (net 2))
+  (segment (start 78.45 95.11001) (end 78.45 100.9) (width 1) (layer B.Cu) (net 2))
+  (segment (start 95.125 103.225) (end 96.95 101.4) (width 1) (layer B.Cu) (net 2))
+  (segment (start 78.45 100.9) (end 80.775 103.225) (width 1) (layer B.Cu) (net 2))
+  (segment (start 109.0556 93.85) (end 104.075 93.85) (width 0.8) (layer B.Cu) (net 2))
+  (segment (start 109.637701 94.432101) (end 109.0556 93.85) (width 0.8) (layer B.Cu) (net 2))
+  (segment (start 111.4806 96.275) (end 110.4377 95.2321) (width 1) (layer B.Cu) (net 2))
+  (segment (start 114.324999 96.275) (end 111.4806 96.275) (width 1) (layer B.Cu) (net 2))
+  (segment (start 101.2 93.85) (end 100.525 94.525) (width 0.8) (layer B.Cu) (net 2))
+  (segment (start 104.075 93.85) (end 101.2 93.85) (width 0.8) (layer B.Cu) (net 2))
+  (segment (start 100.525 94.525) (end 99.825 94.525) (width 0.8) (layer B.Cu) (net 2))
+  (segment (start 99.825 94.525) (end 98.55 95.8) (width 0.8) (layer B.Cu) (net 2))
+  (segment (start 98.55 95.8) (end 98.55 96.4) (width 0.8) (layer B.Cu) (net 2))
+  (segment (start 97.25 97.7) (end 98.55 96.4) (width 0.8) (layer B.Cu) (net 2))
+  (segment (start 96.95 97.7) (end 97.25 97.7) (width 0.8) (layer B.Cu) (net 2))
+  (segment (start 96.95 101.4) (end 96.95 97.7) (width 1) (layer B.Cu) (net 2))
   (segment (start 129.445 72.595) (end 129.445 70.195) (width 1) (layer B.Cu) (net 3) (status 20))
   (segment (start 131.515 74.665) (end 129.445 72.595) (width 1) (layer B.Cu) (net 3))
@@
   (segment (start 105.35001 75.434608) (end 105.324989 75.409587) (width 1) (layer B.Cu) (net 23))
   (segment (start 85.565188 96.575) (end 93.879654 96.575) (width 1) (layer B.Cu) (net 23))
-  (segment (start 105.35001 85.02499) (end 105.35001 75.434608) (width 1) (layer B.Cu) (net 23))
   (segment (start 93.879654 96.575) (end 96.025 94.429654) (width 1) (layer B.Cu) (net 23))
   (segment (start 105.324989 59.950011) (end 105.650511 59.624489) (width 1) (layer B.Cu) (net 23))
   (segment (start 96.025 94.429654) (end 96.025 88.694998) (width 1) (layer B.Cu) (net 23))
-  (segment (start 103.05 87.325) (end 105.35001 85.02499) (width 1) (layer B.Cu) (net 23))
   (segment (start 105.650511 59.624489) (end 106.65 58.625) (width 1) (layer B.Cu) (net 23))
   (segment (start 96.025 88.694998) (end 97.394998 87.325) (width 1) (layer B.Cu) (net 23))
-  (segment (start 97.394998 87.325) (end 103.05 87.325) (width 1) (layer B.Cu) (net 23))
   (segment (start 106.625 58.6) (end 106.65 58.625) (width 1) (layer F.Cu) (net 23))
   (segment (start 106.625 50.9) (end 106.625 58.6) (width 1) (layer F.Cu) (net 23))
+  (segment (start 105.35001 76.229412) (end 105.35001 82.17499) (width 1) (layer B.Cu) (net 23))
+  (segment (start 105.324989 75.409587) (end 105.324989 76.204391) (width 1) (layer B.Cu) (net 23))
+  (segment (start 105.324989 76.204391) (end 105.35001 76.229412) (width 1) (layer B.Cu) (net 23))
+  (segment (start 100.2 87.325) (end 97.394998 87.325) (width 1) (layer B.Cu) (net 23))
+  (segment (start 105.35001 82.17499) (end 100.2 87.325) (width 1) (layer B.Cu) (net 23))
   (segment (start 126.516998 56.555) (end 125.365 56.555) (width 1) (layer B.Cu) (net 24) (status 20))
   (segment (start 127.25363 55.818368) (end 126.516998 56.555) (width 1) (layer B.Cu) (net 24))
@@
   (segment (start 127.325 42.355) (end 129.225 44.255) (width 1) (layer B.Cu) (net 28) (status 20))
   (segment (start 125.475 42.355) (end 127.325 42.355) (width 1) (layer B.Cu) (net 28) (status 10))
+  (segment (start 67.59999 91.99999) (end 70.31501 94.71501) (width 3) (layer B.Cu) (net 29))
   (segment (start 71.6 47.975) (end 71.6 54.720998) (width 3) (layer B.Cu) (net 29))
   (segment (start 71.6 54.720998) (end 67.72499 58.596008) (width 3) (layer B.Cu) (net 29))
@@
   (segment (start 73.075 70.55) (end 77.075001 74.550001) (width 1) (layer B.Cu) (net 29))
   (segment (start 101.325 63.475) (end 101.425 63.375) (width 1) (layer B.Cu) (net 30) (status 30))
-  (segment (start 101.325 67.675) (end 101.325 63.475) (width 1) (layer B.Cu) (net 30) (status 30))
   (segment (start 101.3 68.975) (end 101.3 74.725) (width 1) (layer B.Cu) (net 30))
   (segment (start 101.3 74.725) (end 103.55 76.975) (width 1) (layer B.Cu) (net 30))
@@
   (segment (start 96.158002 50.85) (end 94.154654 50.85) (width 1) (layer B.Cu) (net 30))
   (segment (start 94.154654 50.85) (end 93.604654 50.3) (width 1) (layer B.Cu) (net 30))
+  (segment (start 101.3 62.8) (end 101.375 62.725) (width 0.8) (layer B.Cu) (net 30))
+  (segment (start 101.3 68.975) (end 101.3 62.8) (width 0.8) (layer B.Cu) (net 30))
   (segment (start 73.5 86.982234) (end 73.5 90.90999) (width 3) (layer B.Cu) (net 31))
   (segment (start 71.525 86.775) (end 73.292766 86.775) (width 3) (layer B.Cu) (net 31))
@@
   (segment (start 108.75 86.05) (end 108.75 89.575) (width 1) (layer B.Cu) (net 32) (status 20))
   (segment (start 110.525 84.275) (end 108.75 86.05) (width 1) (layer B.Cu) (net 32) (status 10))
-  (segment (start 102.116999 90.174999) (end 108.82999 90.174999) (width 1) (layer B.Cu) (net 32))
-  (segment (start 98.925 90.335) (end 101.956998 90.335) (width 1) (layer B.Cu) (net 32))
-  (segment (start 101.956998 90.335) (end 102.116999 90.174999) (width 1) (layer B.Cu) (net 32))
+  (segment (start 104.416998 86.05) (end 108.75 86.05) (width 1) (layer B.Cu) (net 32))
+  (segment (start 100.131998 90.335) (end 104.416998 86.05) (width 1) (layer B.Cu) (net 32))
+  (segment (start 98.925 90.335) (end 100.131998 90.335) (width 1) (layer B.Cu) (net 32))
   (zone (net 1) (net_name GND) (layer B.Cu) (hatch edge 0.508)
     (connect_pads (clearance 0.3))
