File: TPFINAL2NOV19/DriverConSensor.sch (KiCad schematic (older format))
At the start: 51 parts, among them J1 PULS1, J2 PULS2, J3 MotorT2, J4 MotorT1, J5 VIn+12, J6 Contac12V, J7 GND, K1 Switch de Encendido, K2 FRS10CS10-12V, K3 FRS10CS10-12V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

Commit message: PCB_casi_listo3
Changed lines of the file:
@@
 Wire Wire Line
 	10800 3700 10800 3800
-Text Label 8900 3250 2    50   ~ 0
+Text Label 8900 1600 2    50   ~ 0
 Relay2y3_NA
 Wire Wire Line
@@
 Relay de encendido\n
 Wire Wire Line
-	8150 2200 8150 2800
-Wire Wire Line
-	8150 2800 7450 2800
-Wire Wire Line
-	8900 2600 8900 3250
-Wire Wire Line
 	4750 2600 4750 3000
 Wire Wire Line
@@
 $EndComp
 Wire Wire Line
-	8150 2200 8600 2200
-Wire Wire Line
 	7750 4850 7750 5200
 Wire Wire Line
@@
 $EndComp
 $Comp
-L power:+12V #PWR?
+L power:+12V #PWR0102
 U 1 1 5DD20DF5
-P 8600 1900
-F 0 "#PWR?" H 8600 1750 50  0001 C CNN
-F 1 "+12V" H 8600 2050 50  0000 C CNN
-F 2 "" H 8600 1900 50  0001 C CNN
-F 3 "" H 8600 1900 50  0001 C CNN
-	1    8600 1900
-	1    0    0    -1
-$EndComp
-Wire Wire Line
-	8600 1900 8600 2200
-Connection ~ 8600 2200
-Wire Wire Line
-	8600 2200 9100 2200
+P 8300 2500
+F 0 "#PWR0102" H 8300 2350 50  0001 C CNN
+F 1 "+12V" H 8300 2650 50  0000 C CNN
+F 2 "" H 8300 2500 50  0001 C CNN
+F 3 "" H 8300 2500 50  0001 C CNN
+	1    8300 2500
+	1    0    0    -1
+$EndComp
+Wire Wire Line
+	8300 2500 8300 2800
+Wire Wire Line
+	8900 2800 8900 2600
+Wire Wire Line
+	7450 2800 8300 2800
+Wire Wire Line
+	9100 2200 8900 2200
+Wire Wire Line
+	8900 2200 8900 1600
+Connection ~ 8300 2800
+Wire Wire Line
+	8300 2800 8900 2800
 $EndSCHEMATC

Commit message: PCB_casi_listo4
Parts:
- C3, C6, C9: footprint Capacitor_THT:C_Disc_D3.8mm_W2.6mm_P2.50mm -> Capacitor_THT:C_Disc_D5.0mm_W2.5mm_P5.00mm
Changed lines of the file:
@@
 F 0 "C9" V 9600 2950 50  0000 L CNN
 F 1 "102" V 9865 2955 50  0000 L CNN
-F 2 "Capacitor_THT:C_Disc_D3.8mm_W2.6mm_P2.50mm" H 9788 2850 50  0001 C CNN
+F 2 "Capacitor_THT:C_Disc_D5.0mm_W2.5mm_P5.00mm" H 9788 2850 50  0001 C CNN
 F 3 "~" H 9750 3000 50  0001 C CNN
 	1    9750 3000
@@
 F 0 "C6" H 5200 1500 50  0000 L CNN
 F 1 "104" H 5250 1400 50  0000 L CNN
-F 2 "Capacitor_THT:C_Disc_D3.8mm_W2.6mm_P2.50mm" H 5138 1250 50  0001 C CNN
+F 2 "Capacitor_THT:C_Disc_D5.0mm_W2.5mm_P5.00mm" H 5138 1250 50  0001 C CNN
 F 3 "~" H 5100 1400 50  0001 C CNN
 	1    5100 1400
@@
 F 0 "C3" H 3100 2950 50  0000 L CNN
 F 1 "104" H 3100 2750 50  0000 L CNN
-F 2 "Capacitor_THT:C_Disc_D3.8mm_W2.6mm_P2.50mm" H 3138 2700 50  0001 C CNN
+F 2 "Capacitor_THT:C_Disc_D5.0mm_W2.5mm_P5.00mm" H 3138 2700 50  0001 C CNN
 F 3 "~" H 3100 2850 50  0001 C CNN
 	1    3100 2850

Commit message: PCB
Parts:
- K1, K2, K3: footprint Relay_THT:Relay_SPDT_SANYOU_SRD_Series_Form_C -> Relay_THT:Relay_SPDT_Omron-G5LE-1
Changed lines of the file:
@@
 Text Notes 6750 3300 0    50   ~ 0
 Activa todo el dispositivo, \npermitiendo alimentar \nlas proximas  etapas\n con los 12v
-$Comp
-L Relay:SANYOU_SRD_Form_C K1
-U 1 1 5E2FB020
-P 7150 2500
-F 0 "K1" V 6550 2500 50  0000 C CNN
-F 1 "Switch de Encendido" V 6650 2550 50  0000 C CNN
-F 2 "Relay_THT:Relay_SPDT_SANYOU_SRD_Series_Form_C" H 7600 2450 50  0001 L CNN
-F 3 "http://www.sanyourelay.ca/public/products/pdf/SRD.pdf" H 7150 2500 50  0001 C CNN
-	1    7150 2500
-	0    1    1    0
-$EndComp
 Text Notes 3750 3700 0    50   ~ 0
 El Pic por un lado mueve el motor hacia \nun lado u hacia el otro según las entradas\nen pulsador 1 o pulsador 2, y segun el \nsensor de corriente lo frena enviando\nlas señales correspondiente a las \nbases de los transistores.\n
@@
 F 0 "K2" H 4550 6000 50  0000 C CNN
 F 1 "FRS10CS10-12V" H 4300 6150 50  0000 C CNN
-F 2 "Relay_THT:Relay_SPDT_SANYOU_SRD_Series_Form_C" H 5050 5600 50  0001 L CNN
+F 2 "Relay_THT:Relay_SPDT_Omron-G5LE-1" H 5050 5600 50  0001 L CNN
 F 3 "http://www.sanyourelay.ca/public/products/pdf/SRD.pdf" H 4600 5650 50  0001 C CNN
 	1    4600 5650
@@
 F 0 "K3" H 2650 5300 50  0000 C CNN
 F 1 "FRS10CS10-12V" H 2900 5150 50  0000 C CNN
-F 2 "Relay_THT:Relay_SPDT_SANYOU_SRD_Series_Form_C" H 3050 5600 50  0001 L CNN
+F 2 "Relay_THT:Relay_SPDT_Omron-G5LE-1" H 3050 5600 50  0001 L CNN
 F 3 "http://www.sanyourelay.ca/public/products/pdf/SRD.pdf" H 2600 5650 50  0001 C CNN
 	1    2600 5650
@@
 Wire Wire Line
 	8300 2800 8900 2800
+$Comp
+L Relay:SANYOU_SRD_Form_C K1
+U 1 1 5E2FB020
+P 7150 2500
+F 0 "K1" V 6550 2500 50  0000 C CNN
+F 1 "Switch de Encendido" V 6650 2550 50  0000 C CNN
+F 2 "Relay_THT:Relay_SPDT_Omron-G5LE-1" H 7600 2450 50  0001 L CNN
+F 3 "http://www.sanyourelay.ca/public/products/pdf/SRD.pdf" H 7150 2500 50  0001 C CNN
+	1    7150 2500
+	0    1    1    0
+$EndComp
 $EndSCHEMATC

Commit message: PCB
Parts:
- U1: CDigikey (none) -> PIC12F675-I/P-ND
Changed lines of the file:
@@
 F 2 "Package_DIP:DIP-8_W7.62mm" H 4550 3150 50  0001 C CNN
 F 3 "http://ww1.microchip.com/downloads/en/DeviceDoc/41190G.pdf" H 3950 2500 50  0001 C CNN
+F 4 "PIC12F675-I/P-ND" H 3950 2500 50  0001 C CNN "CDigikey"
 	1    3950 2500
 	1    0    0    -1

Commit message: PCB_Final
Connections:
- wire segments 187 -> 185
Other:
- note added: "Si ambos Relay están en GND (Normal Cerrado) \nestán desactivados los bornes del motor.\n En cuanto se activa uno (12V) el otro \npermanece desactivado(GND) por lo tanto \nla activacion de cada uno depende del PIN \n2 y 3 respectivamente del PIC\nel motor gira en una dirección y vicecersa \npara cambiar de dirección."
- note removed: "Si ambos Relay están en GND (Normal Cerrado) \nestán desactivados los bornes del motor.\n En cuanto se activa uno (12V) el otro \npermanece desactivado(GND) por lo tanto \nel motor gira en una dirección y vicecersa \npara cambiar de dirección."
Changed lines of the file:
@@
 $EndDescr
-Wire Wire Line
-	6300 2700 6300 1750
 Wire Wire Line
 	7750 1850 7750 1750
@@
 	7600 5200 7600 5450
 $Comp
-L power:+12V #PWR0101
-U 1 1 5D96731E
-P 7200 5050
-F 0 "#PWR0101" H 7200 4900 50  0001 C CNN
-F 1 "+12V" H 7200 5200 50  0000 C CNN
-F 2 "" H 7200 5050 50  0001 C CNN
-F 3 "" H 7200 5050 50  0001 C CNN
-	1    7200 5050
-	1    0    0    -1
-$EndComp
-Wire Wire Line
-	7200 5050 7200 5200
-Wire Wire Line
-	7200 5200 7600 5200
-$Comp
 L power:GND #PWR020
 U 1 1 5D98E2ED
@@
 $EndComp
 Text Notes 5050 7400 0    47   ~ 0
-Si ambos Relay están en GND (Normal Cerrado) \nestán desactivados los bornes del motor.\n En cuanto se activa uno (12V) el otro \npermanece desactivado(GND) por lo tanto \nel motor gira en una dirección y vicecersa \npara cambiar de dirección.
+Si ambos Relay están en GND (Normal Cerrado) \nestán desactivados los bornes del motor.\n En cuanto se activa uno (12V) el otro \npermanece desactivado(GND) por lo tanto \nla activacion de cada uno depende del PIN \n2 y 3 respectivamente del PIC\nel motor gira en una dirección y vicecersa \npara cambiar de dirección.
 Text Notes 1550 7350 0    39   ~ 0
 El código activa o \ndesactiva los \nrelay
@@
 L power:+12V #PWR0102
 U 1 1 5DD20DF5
-P 8300 2500
-F 0 "#PWR0102" H 8300 2350 50  0001 C CNN
-F 1 "+12V" H 8300 2650 50  0000 C CNN
-F 2 "" H 8300 2500 50  0001 C CNN
-F 3 "" H 8300 2500 50  0001 C CNN
-	1    8300 2500
-	1    0    0    -1
-$EndComp
-Wire Wire Line
-	8300 2500 8300 2800
+P 6100 2150
+F 0 "#PWR0102" H 6100 2000 50  0001 C CNN
+F 1 "+12V" H 6100 2300 50  0000 C CNN
+F 2 "" H 6100 2150 50  0001 C CNN
+F 3 "" H 6100 2150 50  0001 C CNN
+	1    6100 2150
+	1    0    0    -1
+$EndComp
 Wire Wire Line
 	8900 2800 8900 2600
 Wire Wire Line
-	7450 2800 8300 2800
-Wire Wire Line
 	9100 2200 8900 2200
 Wire Wire Line
 	8900 2200 8900 1600
-Connection ~ 8300 2800
-Wire Wire Line
-	8300 2800 8900 2800
 $Comp
 L Relay:SANYOU_SRD_Form_C K1
@@
 	0    1    1    0
 $EndComp
+Wire Wire Line
+	7450 2800 8900 2800
+Wire Wire Line
+	6300 2700 6300 1750
+Wire Wire Line
+	6300 2700 6100 2700
+Wire Wire Line
+	6100 2700 6100 2150
+Connection ~ 6300 2700
 $EndSCHEMATC
